File: Chameleon v1_0.kicad_sch (KiCad schematic)
At the start: 203 parts, among them J1 USB_C_Receptacle_USB2.0, SW1 ESC/~, SW10 9, SW11 9, SW12 9, SW13 TAB, SW14 Q, SW15 W, SW16 E, SW17 R, SW18 T, SW19 Y, SW2 1, SW20 U, SW21 I, SW22 O, SW23 O, SW24 O, SW25 STEPPED, SW26 A, SW27 S, SW28 D, SW29 F, SW3 2, SW30 G, SW31 H, SW32 J, SW33 K, SW34 L, SW35 L, SW36 L, SW37 ISO, SW38 >, SW39 Z, SW4 3, SW40 X, SW41 C, SW42 V, SW43 B, SW44 1x2u, SW44 2x2u, SW44 N, SW45 M, SW46 <, SW47 <, SW48 <, SW5 4, SW6 5, SW7 6, SW8 7, SW9 8, U2 W25Q32JVUUIQ, U3 RP2040, U3 SPX3819M5-L-3-3/TR, U4 SN74LV1T34DBV, U5 SRV05-4, Y1 TXM12M0004252LBCEO00T

Commit message: prototype
Tweaked to (probably) prototype status
Parts:
- added SW67, SW68: SW_Push, Keyboard Common:YTSA010, symbol Switch:SW_Push
- ENC1, ENC2, ENC3, ENC4, ENC5, ENC6: footprint Keyboard Encoders:Encoder_Alps_EC11E_Offset_pad -> Keyboard Encoders:Encoder_Alps_EC11E_Small
- H1, H10, H2, H3, H4, H5, H6, H7, H8, H9: now left out of the parts list
- SW1: value ESC/~ -> ~; footprint Keyboard Switches:SW_MX_HotSwap -> Keyboard Switches:SW_MX_HotSwap_FOR ENCODER; symbol Keyboard Switches & Encoders:SW_Push -> Keyboard Switches:SW_Push_GND
- SW10, SW11: value 9 -> ~; symbol Keyboard Switches & Encoders:SW_Push -> Switch:SW_Push
- SW12: value 9 -> ~; footprint Keyboard Switches:SW_MX_HotSwap -> Keyboard Switches:SW_MX_HotSwap_FOR ENCODER; symbol Keyboard Switches & Encoders:SW_Push -> Keyboard Switches:SW_Push_GND
- SW13: value TAB -> ~; symbol Keyboard Switches & Encoders:SW_Push -> Switch:SW_Push
- SW14: value Q -> ~; symbol Keyboard Switches & Encoders:SW_Push -> Switch:SW_Push
- SW15: value W -> ~; symbol Keyboard Switches & Encoders:SW_Push -> Switch:SW_Push
- SW16: value E -> ~; symbol Keyboard Switches & Encoders:SW_Push -> Switch:SW_Push
- SW17: value R -> ~; symbol Keyboard Switches & Encoders:SW_Push -> Switch:SW_Push
- SW18: value T -> ~; symbol Keyboard Switches & Encoders:SW_Push -> Switch:SW_Push
- SW19: value Y -> ~; symbol Keyboard Switches & Encoders:SW_Push -> Switch:SW_Push
- SW2: value 1 -> ~; symbol Keyboard Switches & Encoders:SW_Push -> Switch:SW_Push
- SW20: value U -> ~; symbol Keyboard Switches & Encoders:SW_Push -> Switch:SW_Push
- SW21: value I -> ~; symbol Keyboard Switches & Encoders:SW_Push -> Switch:SW_Push
- SW22, SW23, SW24: value O -> ~; symbol Keyboard Switches & Encoders:SW_Push -> Switch:SW_Push
- SW25: value STEPPED -> ~; footprint Keyboard Switches:SW_MX_HotSwap -> Keyboard Switches:SW_MX_HotSwap_FOR ENCODER; symbol Keyboard Switches & Encoders:SW_Push -> Keyboard Switches:SW_Push_GND
- SW26: value A -> ~; symbol Keyboard Switches & Encoders:SW_Push -> Switch:SW_Push
- SW27: value S -> ~; symbol Keyboard Switches & Encoders:SW_Push -> Switch:SW_Push
- SW28: value D -> ~; symbol Keyboard Switches & Encoders:SW_Push -> Switch:SW_Push
- SW29: value F -> ~; symbol Keyboard Switches & Encoders:SW_Push -> Switch:SW_Push
- SW3: value 2 -> ~; symbol Keyboard Switches & Encoders:SW_Push -> Switch:SW_Push
- SW30: value G -> ~; symbol Keyboard Switches & Encoders:SW_Push -> Switch:SW_Push
- SW31: value H -> ~; symbol Keyboard Switches & Encoders:SW_Push -> Switch:SW_Push
- SW32: value J -> ~; symbol Keyboard Switches & Encoders:SW_Push -> Switch:SW_Push
- SW33: value K -> ~; symbol Keyboard Switches & Encoders:SW_Push -> Switch:SW_Push
- SW34, SW35: value L -> ~; symbol Keyboard Switches & Encoders:SW_Push -> Switch:SW_Push
- SW36: value L -> ~; footprint Keyboard Switches:SW_MX_HotSwap -> Keyboard Switches:SW_MX_HotSwap_FOR ENCODER; symbol Keyboard Switches & Encoders:SW_Push -> Keyboard Switches:SW_Push_GND
- SW37: value ISO -> ~; footprint Keyboard Switches:SW_MX_HotSwap -> Keyboard Switches:SW_MX_HotSwap_FOR ENCODER; symbol Keyboard Switches & Encoders:SW_Push -> Keyboard Switches:SW_Push_GND
- SW38: value > -> ~; symbol Keyboard Switches & Encoders:SW_Push -> Switch:SW_Push
- SW39: value Z -> ~; symbol Keyboard Switches & Encoders:SW_Push -> Switch:SW_Push
- SW4: value 3 -> ~; symbol Keyboard Switches & Encoders:SW_Push -> Switch:SW_Push
- SW40: value X -> ~; symbol Keyboard Switches & Encoders:SW_Push -> Switch:SW_Push
- SW41: value C -> ~; symbol Keyboard Switches & Encoders:SW_Push -> Switch:SW_Push
- SW42: value V -> ~; symbol Keyboard Switches & Encoders:SW_Push -> Switch:SW_Push
- SW43: value B -> ~; symbol Keyboard Switches & Encoders:SW_Push -> Switch:SW_Push
- SW44: value 2x2u -> ~; symbol Keyboard Switches & Encoders:SW_Push -> Switch:SW_Push
- SW44: value 1x2u -> ~; symbol Keyboard Switches & Encoders:SW_Push -> Switch:SW_Push
- SW44: value N -> ~; symbol Keyboard Switches & Encoders:SW_Push -> Switch:SW_Push
- SW45: value M -> ~; symbol Keyboard Switches & Encoders:SW_Push -> Switch:SW_Push
- SW46, SW47: value < -> ~; symbol Keyboard Switches & Encoders:SW_Push -> Switch:SW_Push
- SW48: value < -> ~; footprint Keyboard Switches:SW_MX_HotSwap -> Keyboard Switches:SW_MX_HotSwap_FOR ENCODER; symbol Keyboard Switches & Encoders:SW_Push -> Keyboard Switches:SW_Push_GND
- SW5: value 4 -> ~; symbol Keyboard Switches & Encoders:SW_Push -> Switch:SW_Push
- SW6: value 5 -> ~; symbol Keyboard Switches & Encoders:SW_Push -> Switch:SW_Push
- SW7: value 6 -> ~; symbol Keyboard Switches & Encoders:SW_Push -> Switch:SW_Push
- SW8: value 7 -> ~; symbol Keyboard Switches & Encoders:SW_Push -> Switch:SW_Push
- SW9: value 8 -> ~; symbol Keyboard Switches & Encoders:SW_Push -> Switch:SW_Push
Connections:
- net Col_0: now also ENC3.S1, ENC4.S1, ENC5.S1, ENC6.S1, U3.18 (GPIO15); no longer ENC3.S2, ENC4.S2, ENC5.S2, ENC6.S2, U3.38 (GPIO26_ADC0)
- net Col_1: now also U3.17 (GPIO14); no longer U3.37 (GPIO25)
- net Col_2: now also U3.8 (GPIO6); no longer U3.17 (GPIO14)
- net Col_3: now also U3.7 (GPIO5); no longer U3.16 (GPIO13)
- net Col_4: now also U3.6 (GPIO4); no longer U3.15 (GPIO12)
- net Col_5: now also U3.5 (GPIO3); no longer U3.14 (GPIO11)
- net ENC1_A: now also U3.29 (GPIO18); no longer U3.39 (GPIO27_ADC1)
- net ENC1_B: now also U3.30 (GPIO19); no longer U3.40 (GPIO28_ADC2)
- net ENC2_A: now also U3.39 (GPIO27_ADC1); no longer U3.6 (GPIO4)
- net ENC2_B: now also U3.2 (GPIO0); no longer U3.7 (GPIO5)
- net ENC3: now also ENC3.S2; no longer ENC3.S1
- net ENC3_A: now also C21.2, ENC3.B, ENC5.B, U3.28 (GPIO17); no longer C20.1, ENC3.A, ENC5.A, U3.32 (GPIO21)
- net ENC3_B: now also C20.1, ENC3.A, ENC5.A, U3.27 (GPIO16); no longer C21.2, ENC3.B, ENC5.B, U3.31 (GPIO20)
- net ENC4: now also ENC4.S2; no longer ENC4.S1
- net ENC4_A: now also C23.2, ENC4.B, ENC6.B, U3.13 (GPIO10); no longer C22.1, ENC4.A, ENC6.A, U3.9 (GPIO7)
- net ENC4_B: now also C22.1, ENC4.A, ENC6.A, U3.12 (GPIO9); no longer C23.2, ENC4.B, ENC6.B, U3.8 (GPIO6)
- net ENC5: now also ENC5.S2; no longer ENC5.S1
- net ENC6: now also ENC6.S2; no longer ENC6.S1
- net GND: now also SW1.3, SW12.3, SW25.3, SW36.3, SW37.3, SW48.3, SW67.1, SW68.1
- net RGB: now also U3.31 (GPIO20); no longer U3.41 (GPIO29_ADC3)
- net Row_0: now also U3.41 (GPIO29_ADC3); no longer U3.2 (GPIO0)
- net Row_1: now also U3.34 (GPIO22); no longer U3.4 (GPIO2)
- net Row_2: now also U3.32 (GPIO21); no longer U3.3 (GPIO1)
- net Row_3: now also U3.36 (GPIO24); no longer U3.5 (GPIO3)
- net Row_4: now also U3.16 (GPIO13); no longer U3.30 (GPIO19)
- net Row_5: now also U3.3 (GPIO1); no longer U3.13 (GPIO10)
- net Row_6: now also U3.14 (GPIO11); no longer U3.29 (GPIO18)
- net Row_7: now also U3.4 (GPIO2); no longer U3.12 (GPIO9)
- net Row_8: now also U3.15 (GPIO12); no longer U3.28 (GPIO17)
- net at RGB5.1 (DOUT), RGB6.3 (DIN): no longer RGB10.3 (DIN), RGB9.1 (DOUT)
- net at RGB10.1 (DOUT), RGB11.3 (DIN): no longer RGB6.1 (DOUT), RGB7.3 (DIN)
- net at RGB12.1 (DOUT): no longer RGB8.1 (DOUT)
- net at RGB11.1 (DOUT), RGB12.3 (DIN): no longer RGB7.1 (DOUT), RGB8.3 (DIN)
- net BOOT: no longer names the net of R6.2
- net BOOT: now also SW68.2
- net RESET: no longer names the net of R8.2, U3.26 (RUN)
- net RESET: now also SW67.2
- new net: RGB10.3 (DIN), RGB9.1 (DOUT)
- new net: RGB7.1 (DOUT), RGB8.3 (DIN)
- new net: RGB6.1 (DOUT), RGB7.3 (DIN)
- no-connect marks 12 -> 14
Other:
- moved on the sheet: C1, C10, C11, C12, C13, C14, C15, C16, C17, C18, C19, C2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
