File: Chameleon/Plate/v1.10/Chameleon Plate v1_10.kicad_pcb (KiCad board)
At the start: 2 copper layers, 228 x 93 mm, 66 parts

Commit message: Skinny Chameleon
v1.00
Parts:
- moved SW14 5.00 mm to (66.2, 73.0)
- moved SW2 5.00 mm to (66.2, 54.0)
- moved SW26 5.00 mm to (66.2, 92.1)
- moved SW38 5.00 mm to (66.2, 111.1)
- moved SW50 5.00 mm to (66.2, 130.2)
- moved H1 5.00 mm to (56.7, 82.6)
- moved H2 5.00 mm to (56.7, 120.7)
- moved H3 5.00 mm to (151.9, 101.6)
- moved H4 5.00 mm to (247.2, 82.6)
- moved H5 5.00 mm to (247.2, 120.7)
- moved H6 5.00 mm to (56.7, 63.5)
- moved H7 5.00 mm to (247.2, 63.5)
- moved SW1 5.00 mm to (47.1, 54.0)
- moved SW10 5.00 mm to (218.6, 54.0)
- moved SW11 5.00 mm to (237.6, 54.0)
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Other:
- outline, holes or cut-outs redrawn
