File: Skinny Chameleon/v1.10/Skinny Chameleon.kicad_sch (KiCad schematic)
At the start: 206 parts, among them SW10 PG151101S11, SW11 PG151101S11, SW13 PG151101S11, SW14 PG151101S11, SW15 PG151101S11, SW16 PG151101S11, SW17 PG151101S11, SW18 PG151101S11, SW19 PG151101S11, SW2 PG151101S11, SW20 PG151101S11, SW21 PG151101S11, SW22 PG151101S11, SW23 PG151101S11, SW24 PG151101S11, SW26 PG151101S11, SW27 PG151101S11, SW28 PG151101S11, SW29 PG151101S11, SW3 PG151101S11, SW30 PG151101S11, SW31 PG151101S11, SW32 PG151101S11, SW33 PG151101S11, SW34 PG151101S11, SW35 PG151101S11, SW38 PG151101S11, SW39 PG151101S11, SW4 PG151101S11, SW40 PG151101S11, SW41 PG151101S11, SW42 PG151101S11, SW43 PG151101S11, SW44 PG151101S11, SW45 PG151101S11, SW46 PG151101S11, SW47 PG151101S11, SW5 PG151101S11, SW6 PG151101S11, SW67 YTSA010, SW68 YTSA010, SW7 PG151101S11, SW8 PG151101S11, SW9 PG151101S11, U2 W25Q32JVUUIQ, U3 RP2040, U3 SPX3819M5-L-3-3/TR, U4 SN74LV1T34DBV, U5 SRV05-4, Y1 TXM12M0004252LBCEO00T

Commit message: Skinny Chamelelon v1.10
- Updated Planck Mounting holes
- Updated centering on USB (was centered on 19.05 spacing?)
Parts:
- Logo2: footprint Logotypes:Powered_by_QMK -> Logotypes:qmk logo
Changed lines of the file:
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@@
 	(title_block
 		(title "Skinny Chameleon")
-		(date "2024-06-04")
+		(date "2024-08-16")
 		(rev "v1.10")
 		(company "Tweety's Wild Thinking")
@@
 			)
 		)
-		(property "Footprint" "Logotypes:Powered_by_QMK"
+		(property "Footprint" "Logotypes:qmk logo"
 			(at 24.13 267.97 0)
 			(effects
