File: Chameleon/PCB/v1.20/Chameleon.kicad_pcb (KiCad board)
At the start: 2 copper layers, 226 x 92 mm, 205 parts, among them SW10 PG151101S11, SW11 PG151101S11, SW13 PG151101S11, SW14 PG151101S11, SW15 PG151101S11, SW16 PG151101S11, SW17 PG151101S11, SW18 PG151101S11, SW19 PG151101S11, SW2 PG151101S11, SW20 PG151101S11, SW21 PG151101S11, SW22 PG151101S11, SW23 PG151101S11, SW24 PG151101S11, SW25 PG151101S11, SW26 PG151101S11, SW27 PG151101S11, SW28 PG151101S11, SW29 PG151101S11, SW3 PG151101S11, SW30 PG151101S11, SW31 PG151101S11, SW32 PG151101S11, SW33 PG151101S11, SW34 PG151101S11, SW35 PG151101S11, SW36 PG151101S11, SW38 PG151101S11, SW39 PG151101S11, SW4 PG151101S11, SW40 PG151101S11, SW41 PG151101S11, SW42 PG151101S11, SW43 PG151101S11, SW44 PG151101S11, SW45 PG151101S11, SW46 PG151101S11, SW47 PG151101S11, SW5 PG151101S11, SW50 PG151101S11, SW51 PG151101S11, SW52 PG151101S11, SW53 PG151101S11, SW54 PG151101S11, SW55 PG151101S11, SW56 PG151101S11, SW57 PG151101S11, SW58 PG151101S11, SW59 PG151101S11, SW6 PG151101S11, SW61 PG151101S11, SW62 PG151101S11, SW63 PG151101S11, SW64 PG151101S11, SW65 PG151101S11, SW66 PG151101S11, SW67 YTSA010, SW68 YTSA010, SW7 PG151101S11, SW8 PG151101S11, SW9 PG151101S11, U1 SPX3819M5-L-3-3/TR, U2 W25Q32JVUUIQ, U3 RP2040, U4 SN74LV1T34DBV, U5 SRV05-4, Y1 TXM12M0004252LBCEO00T

Commit message: Chameleon v1.20
Parts:
- removed ENC1, ENC2, ENC3, ENC4, ENC5, ENC6: RotaryEncoder_Switch, Keyboard Encoders:Encoder_Alps_EC11E_Small
- added Logo3: CE, Logotypes:CE, F.Cu at (168.0, 82.4)
- added Logo4: RoHS, Logotypes:RoHs, F.Cu at (156.7, 82.4)
- F1: value CF06V5TR50 -> 0603L050/6AR
- Logo1: footprint Logotypes:CC_BY_SA_40_tiny -> Logotypes:CC_BY_SA_40_line
- SW1, SW12: footprint Keyboard Switches:SW_MX_HotSwap_FOR ENCODER -> Keyboard Switches:SW_MX_HotSwap_Encoder
- SW37, SW48, SW49, SW60: footprint Keyboard Switches:SW_MX_HotSwap_FOR ENCODER -> Keyboard Switches:SW_MX_HotSwap_Encoder_inverted
- moved Logo2 25.3 mm to (103.7, 82.4)
- moved Logo1 23.3 mm to (129.0, 82.6)
- moved C11 4.65 mm to (49.8, 54.5)
- moved C12 4.65 mm to (49.8, 56.3)
- moved U1 4.65 mm to (51.9, 55.3)
- moved D1 3.49 mm to (51.6, 51.8), turned to 180 degrees
- moved D2 2.93 mm to (69.1, 63.5)
- moved U4 2.57 mm to (55.4, 49.0)
- moved F1 1.51 mm to (58.6, 48.2)
- moved U5 1.38 mm to (62.4, 48.4)
- moved R2 1.33 mm to (73.0, 54.8), turned to -90 degrees
- moved USB1 1.12 mm to (70.8, 47.3)
- moved R1 0.86 mm to (69.2, 54.4), turned to 0 degrees
Connections:
- D1 pad 2: ENC1 -> Net-(D1-A)
- D12 pad 2: ENC2 -> Net-(D12-A)
- D37 pad 2: ENC3 -> Net-(D37-A)
- D48 pad 2: ENC4 -> Net-(D48-A)
- D49 pad 2: ENC5 -> Net-(D49-A)
- D60 pad 2: ENC6 -> Net-(D60-A)
- SW1 pad 2: ENC1 -> Net-(D1-A)
- SW12 pad 2: ENC2 -> Net-(D12-A)
- SW37 pad 2: ENC3 -> Net-(D37-A)
- SW48 pad 2: ENC4 -> Net-(D48-A)
- SW49 pad 2: ENC5 -> Net-(D49-A)
- SW60 pad 2: ENC6 -> Net-(D60-A)
Routing:
- net Net-(D48-A): track 0.00 -> 30.1 mm, vias 0 -> 2
- net ENC4: track 30.1 -> 0.00 mm, vias 2 -> 0
- net Net-(D60-A): track 0.00 -> 28.2 mm, vias 0 -> 2
- net ENC6: track 28.2 -> 0.00 mm, vias 2 -> 0
- net Net-(D12-A): track 0.00 -> 25.8 mm, vias 0 -> 2
- net ENC2: track 25.8 -> 0.00 mm, vias 2 -> 0
- net Net-(D49-A): track 0.00 -> 18.8 mm, vias 0 -> 1
- net ENC5: track 18.8 -> 0.00 mm, vias 1 -> 0
- net Net-(D37-A): track 0.00 -> 18.8 mm, vias 0 -> 1
- net ENC3: track 18.8 -> 0.00 mm, vias 1 -> 0
- net ENC1: track 9.41 -> 0.00 mm, vias 1 -> 0
- net Net-(D1-A): track 0.00 -> 8.61 mm, vias 0 -> 1
- net GND: track 9.39 -> 4.78 mm, vias 82 -> 77
- net +3V3: track 86.3 -> 90.4 mm
- net Net-(D2-A): track 2.81 -> 5.74 mm
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Other:
- board text added: "Chameleon - v1.20 - Markus Knutsson 2025 https://github.com/TweetyDaBird"
- board text added: "LEFT"
- board text added: "MIT"
- board text added: "RIGHT"
- board text added: "Warning! - Please support sockets on the backside as you insert a switch to avoid damage to the socket/solder pad!"
- board text removed: "Chameleon - v1.11 - Markus Knutsson 2024 https://github.com/TweetyDaBird"
- board text removed: "The Chameleon PCB supports a 5x12 or 4x12 matrix with 8 RGB LEDs for under-glow and one encoder per corner. Each layout supports a full matrix, a single 2u or two 2u keys on the bottom row. Please note that 2u keys and stabilizers should only be installed at the CURRENT bottom row."
- board text removed: "The bottom corner encoders connect in parallel to the same input, and only ONE encoder per corner is functional at each time. Please do NOT install encoders in both rows! The optional placements for RGB LEDs are parallel, and only ONE bottom row is functional at each time. Please do NOT install LEDs in both bottom rows!"
