File: Chameleon/PCB/v1.20/Chameleon.kicad_sch (KiCad schematic)
At the start: 205 parts, among them SW10 PG151101S11, SW11 PG151101S11, SW13 PG151101S11, SW14 PG151101S11, SW15 PG151101S11, SW16 PG151101S11, SW17 PG151101S11, SW18 PG151101S11, SW19 PG151101S11, SW2 PG151101S11, SW20 PG151101S11, SW21 PG151101S11, SW22 PG151101S11, SW23 PG151101S11, SW24 PG151101S11, SW26 PG151101S11, SW27 PG151101S11, SW28 PG151101S11, SW29 PG151101S11, SW3 PG151101S11, SW30 PG151101S11, SW31 PG151101S11, SW32 PG151101S11, SW33 PG151101S11, SW34 PG151101S11, SW35 PG151101S11, SW38 PG151101S11, SW39 PG151101S11, SW4 PG151101S11, SW40 PG151101S11, SW41 PG151101S11, SW42 PG151101S11, SW43 PG151101S11, SW44 PG151101S11, SW45 PG151101S11, SW46 PG151101S11, SW47 PG151101S11, SW5 PG151101S11, SW6 PG151101S11, SW67 YTSA010, SW68 YTSA010, SW7 PG151101S11, SW8 PG151101S11, SW9 PG151101S11, U2 W25Q32JVUUIQ, U3 RP2040, U3 SPX3819M5-L-3-3/TR, U4 SN74LV1T34DBV, U5 SRV05-4, Y1 TXM12M0004252LBCEO00T

Commit message: Chameleon v1.20
Parts:
- removed ENC1, ENC2, ENC3, ENC4, ENC5, ENC6: RotaryEncoder_Switch, Keyboard Encoders:Encoder_Alps_EC11E_Small, symbol Keyboard Switches:Rotary_Encoder_Click
- removed SW12, SW25, SW36, SW37, SW48: ~, Keyboard Switches:SW_MX_HotSwap_FOR ENCODER, symbol Keyboard Switches:SW_Push_GND
- added Logo3: CE, Logotypes:CE, symbol Logotypes:CC-BY-SA-4.0
- added Logo4: RoHS, Logotypes:RoHs, symbol Logotypes:CC-BY-SA-4.0
- added unit 1 of SW1
- added SW12: ~, Keyboard Switches:SW_MX_HotSwap_Encoder, symbol Keyboard Switches:SW_MX_HotSwap_Encoder
- added SW37, SW48, SW49, SW60: ~, Keyboard Switches:SW_MX_HotSwap_Encoder_inverted, symbol Keyboard Switches:SW_MX_HotSwap_Encoder
- Logo1: footprint Logotypes:CC_BY_SA_40_tiny -> Logotypes:CC_BY_SA_40_line
- SW1: footprint Keyboard Switches:SW_MX_HotSwap_FOR ENCODER -> Keyboard Switches:SW_MX_HotSwap_Encoder; symbol Keyboard Switches:SW_Push_GND -> Keyboard Switches:SW_MX_HotSwap_Encoder; now in the parts list
- SW10, SW11, SW13, SW14, SW15, SW16, SW17, SW18, SW19, SW2, SW20, SW21, SW22, SW23, SW24, SW3, SW4, SW5, SW6, SW7, SW8, SW9: value PG151101S11 -> SW_Push; footprint Keyboard Switches:SW_MX_HotSwap -> (none); LCSC Part # C2803348 -> (none); now not fitted
- SW25: renamed from SW13; value PG151101S11 -> SW_Push; footprint Keyboard Switches:SW_MX_HotSwap -> (none); LCSC Part # C2803348 -> (none); now not fitted
- SW26: renamed from SW14; value PG151101S11 -> SW_Push; footprint Keyboard Switches:SW_MX_HotSwap -> (none); LCSC Part # C2803348 -> (none); now not fitted
- SW27: renamed from SW15; value PG151101S11 -> SW_Push; footprint Keyboard Switches:SW_MX_HotSwap -> (none); LCSC Part # C2803348 -> (none); now not fitted
- SW28: renamed from SW16; value PG151101S11 -> SW_Push; footprint Keyboard Switches:SW_MX_HotSwap -> (none); LCSC Part # C2803348 -> (none); now not fitted
- SW29: renamed from SW17; value PG151101S11 -> SW_Push; footprint Keyboard Switches:SW_MX_HotSwap -> (none); LCSC Part # C2803348 -> (none); now not fitted
- SW30: renamed from SW18; value PG151101S11 -> SW_Push; footprint Keyboard Switches:SW_MX_HotSwap -> (none); LCSC Part # C2803348 -> (none); now not fitted
- SW31: renamed from SW19; value PG151101S11 -> SW_Push; footprint Keyboard Switches:SW_MX_HotSwap -> (none); LCSC Part # C2803348 -> (none); now not fitted
- SW32: renamed from SW20; value PG151101S11 -> SW_Push; footprint Keyboard Switches:SW_MX_HotSwap -> (none); LCSC Part # C2803348 -> (none); now not fitted
- SW33: renamed from SW21; value PG151101S11 -> SW_Push; footprint Keyboard Switches:SW_MX_HotSwap -> (none); LCSC Part # C2803348 -> (none); now not fitted
- SW34: renamed from SW22; value PG151101S11 -> SW_Push; footprint Keyboard Switches:SW_MX_HotSwap -> (none); LCSC Part # C2803348 -> (none); now not fitted
- SW35: renamed from SW23; value PG151101S11 -> SW_Push; footprint Keyboard Switches:SW_MX_HotSwap -> (none); LCSC Part # C2803348 -> (none); now not fitted
- SW36: renamed from SW24; value PG151101S11 -> SW_Push; footprint Keyboard Switches:SW_MX_HotSwap -> (none); LCSC Part # C2803348 -> (none); now not fitted
- SW38: renamed from SW26; value PG151101S11 -> SW_Push; footprint Keyboard Switches:SW_MX_HotSwap -> (none); LCSC Part # C2803348 -> (none); now not fitted
- SW39: renamed from SW27; value PG151101S11 -> SW_Push; footprint Keyboard Switches:SW_MX_HotSwap -> (none); LCSC Part # C2803348 -> (none); now not fitted
- SW40: renamed from SW28; value PG151101S11 -> SW_Push; footprint Keyboard Switches:SW_MX_HotSwap -> (none); LCSC Part # C2803348 -> (none); now not fitted
- SW41: renamed from SW29; value PG151101S11 -> SW_Push; footprint Keyboard Switches:SW_MX_HotSwap -> (none); LCSC Part # C2803348 -> (none); now not fitted
- SW42: renamed from SW30; value PG151101S11 -> SW_Push; footprint Keyboard Switches:SW_MX_HotSwap -> (none); LCSC Part # C2803348 -> (none); now not fitted
- SW43: renamed from SW31; value PG151101S11 -> SW_Push; footprint Keyboard Switches:SW_MX_HotSwap -> (none); LCSC Part # C2803348 -> (none); now not fitted
- SW44: renamed from SW32; value PG151101S11 -> SW_Push; footprint Keyboard Switches:SW_MX_HotSwap -> (none); LCSC Part # C2803348 -> (none); now not fitted
- SW45: renamed from SW33; value PG151101S11 -> SW_Push; footprint Keyboard Switches:SW_MX_HotSwap -> (none); LCSC Part # C2803348 -> (none); now not fitted
- SW46: renamed from SW34; value PG151101S11 -> SW_Push; footprint Keyboard Switches:SW_MX_HotSwap -> (none); LCSC Part # C2803348 -> (none); now not fitted
- SW47: renamed from SW35; value PG151101S11 -> SW_Push; footprint Keyboard Switches:SW_MX_HotSwap -> (none); LCSC Part # C2803348 -> (none); now not fitted
- SW50: renamed from SW38; value PG151101S11 -> SW_Push; footprint Keyboard Switches:SW_MX_HotSwap -> (none); LCSC Part # C2803348 -> (none); now not fitted
- SW51: renamed from SW39; value PG151101S11 -> SW_Push; footprint Keyboard Switches:SW_MX_HotSwap -> (none); LCSC Part # C2803348 -> (none); now not fitted
- SW52: renamed from SW40; value PG151101S11 -> SW_Push; footprint Keyboard Switches:SW_MX_HotSwap -> (none); LCSC Part # C2803348 -> (none); now not fitted
- SW53: renamed from SW41; value PG151101S11 -> SW_Push; footprint Keyboard Switches:SW_MX_HotSwap -> (none); LCSC Part # C2803348 -> (none); now not fitted
- SW54: renamed from SW42; value PG151101S11 -> SW_Push; footprint Keyboard Switches:SW_MX_HotSwap -> (none); LCSC Part # C2803348 -> (none); now not fitted
- SW55: renamed from SW43; value PG151101S11 -> SW_Push; footprint Keyboard Switches:SW_MX_HotSwap -> (none); LCSC Part # C2803348 -> (none); now not fitted
- SW56, SW61, SW62, SW63, SW64, SW65, SW66: renamed from SW44; value PG151101S11 -> SW_Push; footprint Keyboard Switches:SW_MX_HotSwap -> (none); LCSC Part # C2803348 -> (none); now not fitted
- SW57: renamed from SW45; value PG151101S11 -> SW_Push; footprint Keyboard Switches:SW_MX_HotSwap -> (none); LCSC Part # C2803348 -> (none); now not fitted
- SW58: renamed from SW46; value PG151101S11 -> SW_Push; footprint Keyboard Switches:SW_MX_HotSwap -> (none); LCSC Part # C2803348 -> (none); now not fitted
- SW59: renamed from SW47; value PG151101S11 -> SW_Push; footprint Keyboard Switches:SW_MX_HotSwap -> (none); LCSC Part # C2803348 -> (none); now not fitted
- SW67, SW68: value YTSA010 -> SW_Push; footprint Keyboard Common:YTSA010 -> (none); LCSC Part # C967783 -> (none); now not fitted
- renumbered C9 to C1, C8 to C10, C1 to C11, C2 to C12, C5 to C13, C3 to C14, C4 to C15, C10 to C2, C11 to C3, C12 to C4, C13 to C5, C14 to C6, C15 to C7, C6 to C8, C7 to C9, D13 to D25, D14 to D26, D15 to D27, D16 to D28, D17 to D29, D18 to D30, D19 to D31, D20 to D32, D21 to D33, D22 to D34, D23 to D35, D24 to D36, D25 to D37, D26 to D38, D27 to D39, D28 to D40, D29 to D41, D30 to D42, D31 to D43, D32 to D44, D33 to D45, D34 to D46, D35 to D47, D36 to D48, D37 to D49, D38 to D50, D39 to D51, D40 to D52, D41 to D53, D42 to D54, D43 to D55, D44 to D56, D45 to D57, D46 to D58, D47 to D59, D48 to D60, R5 to R10, R8 to R3, R6 to R4, R3 to R5, R4 to R6, U3 to U1
Connections:
- net Col_0: now also SW1.1, SW1.S1, SW12.1, SW12.S1, SW37.1, SW37.S1, SW48.1, SW48.S1, SW49.1, SW49.S1, SW60.1, SW60.S1; no longer SW1.1
- net ENC1_A: now also SW1.A
- net ENC1_B: now also SW1.B
- net ENC2_A: now also SW12.A
- net ENC2_B: now also SW12.B
- net ENC3_A: now also SW37.A, SW49.A
- net ENC3_B: now also SW37.B, SW49.B
- net ENC4_A: now also SW48.A, SW60.A
- net ENC4_B: now also SW48.B, SW60.B
- net GND: now also SW1.C (GND), SW1.MP (GND), SW12.C (GND), SW12.MP (GND), SW37.C (GND), SW37.MP (GND), SW48.C (GND), SW48.MP (GND), SW49.C (GND), SW49.MP (GND), SW60.C (GND), SW60.MP (GND); no longer SW1.3
- net ENC1: no longer names the net of D1.2 (A)
- net ENC1: now also SW1.2, SW1.S2; no longer SW1.2
- net ENC2: no longer names the net of D12.2 (A)
- net ENC2: now also SW12.2, SW12.S2
- net ENC3: no longer names the net of D37.2 (A)
- net ENC3: now also SW37.2, SW37.S2
- net ENC4: no longer names the net of D48.2 (A)
- net ENC4: now also SW48.2, SW48.S2
- net ENC5: no longer names the net of D49.2 (A)
- net ENC5: now also SW49.2, SW49.S2
- net ENC6: no longer names the net of D60.2 (A)
- net ENC6: now also SW60.2, SW60.S2
