File: PCB/v1.20/Chameleon.kicad_pcb (KiCad board)
At the start: 2 copper layers, 226 x 92 mm, 201 parts, among them SW10 PG151101S11, SW11 PG151101S11, SW13 PG151101S11, SW14 PG151101S11, SW15 PG151101S11, SW16 PG151101S11, SW17 PG151101S11, SW18 PG151101S11, SW19 PG151101S11, SW2 PG151101S11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

Commit message: re-ordered files
Parts:
- renumbered SW68 to TACT1, SW67 to TACT2
Routing:
- net Row_4: track 117.8 -> 115.3 mm
