File: PCB/v1.20/Chameleon.kicad_sch (KiCad schematic)
At the start: 201 parts, among them SW10 SW_Push, SW11 SW_Push, SW13 SW_Push, SW14 SW_Push, SW15 SW_Push, SW16 SW_Push, SW17 SW_Push, SW18 SW_Push, SW19 SW_Push, SW2 SW_Push, SW20 SW_Push, SW21 SW_Push, SW22 SW_Push, SW23 SW_Push, SW24 SW_Push, SW25 SW_Push, SW26 SW_Push, SW27 SW_Push, SW28 SW_Push, SW29 SW_Push, SW3 SW_Push, SW30 SW_Push, SW31 SW_Push, SW32 SW_Push, SW33 SW_Push, SW34 SW_Push, SW35 SW_Push, SW36 SW_Push, SW38 SW_Push, SW39 SW_Push, SW4 SW_Push, SW40 SW_Push, SW41 SW_Push, SW42 SW_Push, SW43 SW_Push, SW44 SW_Push, SW45 SW_Push, SW46 SW_Push, SW47 SW_Push, SW5 SW_Push, SW50 SW_Push, SW51 SW_Push, SW52 SW_Push, SW53 SW_Push, SW54 SW_Push, SW55 SW_Push, SW56 SW_Push, SW57 SW_Push, SW58 SW_Push, SW59 SW_Push, SW6 SW_Push, SW61 SW_Push, SW62 SW_Push, SW63 SW_Push, SW64 SW_Push, SW65 SW_Push, SW66 SW_Push, SW67 SW_Push, SW68 SW_Push, SW7 SW_Push, SW8 SW_Push, SW9 SW_Push, U1 SPX3819M5-L-3-3/TR, U2 W25Q32JVUUIQ, U3 RP2040, U4 SN74LV1T34DBV, U5 SRV05-4, Y1 TXM12M0004252LBCEO00T

Commit message: re-ordered files
Parts:
- TACT1: renamed from SW68; value SW_Push -> TACT; LCSC Part # (none) -> C557591; now fitted
- TACT2: renamed from SW67; value SW_Push -> TACT; LCSC Part # (none) -> C557591; now fitted
Changed lines of the file:
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@@
 		(in_bom yes)
 		(on_board yes)
-		(dnp yes)
+		(dnp no)
 		(fields_autoplaced yes)
-		(property "Reference" "SW68"
+		(property "Reference" "TACT1"
 			(at 252.73 80.01 0)
 			(effects
@@
 			)
 		)
-		(property "Value" "SW_Push"
+		(property "Value" "TACT"
 			(at 252.73 82.55 0)
 			(effects
@@
 		)
 		(property "Description" "Push button switch, generic, two pins"
+			(at 252.73 87.63 0)
+			(effects
+				(font
+					(size 1.27 1.27)
+				)
+				(hide yes)
+			)
+		)
+		(property "LCSC Part #" "C557591"
 			(at 252.73 87.63 0)
 			(effects
@@
 			(project "Chameleon v1_11"
 				(path "/9cbb0ce1-ad88-4669-adb0-4b1f4ac042dc"
-					(reference "SW68")
+					(reference "TACT1")
 					(unit 1)
 				)
@@
 		(in_bom yes)
 		(on_board yes)
-		(dnp yes)
+		(dnp no)
 		(fields_autoplaced yes)
-		(property "Reference" "SW67"
+		(property "Reference" "TACT2"
 			(at 293.37 78.74 0)
 			(effects
@@
 			)
 		)
-		(property "Value" "SW_Push"
+		(property "Value" "TACT"
 			(at 293.37 81.28 0)
 			(effects
@@
 		)
 		(property "Description" "Push button switch, generic, two pins"
+			(at 293.37 86.36 0)
+			(effects
+				(font
+					(size 1.27 1.27)
+				)
+				(hide yes)
+			)
+		)
+		(property "LCSC Part #" "C557591"
 			(at 293.37 86.36 0)
 			(effects
@@
 			(project "Chameleon v1_11"
 				(path "/9cbb0ce1-ad88-4669-adb0-4b1f4ac042dc"
-					(reference "SW67")
-					(unit 1)
-				)
+					(reference "TACT2")
+					(unit 1)
+				)
